File: CheckPoint1/KiCad/esquematico/esquematico.kicad_sch (KiCad schematic)
At the start: 31 parts, among them J1 Conn_01x02, J2 Conn_01x02, Q10 TIP32A, Q2 BC547, Q3 BC557, Q4 BC557, Q5 BC547, Q6 BC547, Q7 BC547, Q8 BC547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

Commit message: Funciona
Other:
- company: (none) -> FIUBA - TA138
- title: (none) -> Fuente Regulada con Protección Foldback
Changed lines of the file:
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@@
 	(generator_version "10.0")
 	(paper "A4")
+	(title_block
+		(title "Fuente Regulada con Protección Foldback")
+		(date "2026-04-10")
+		(company "FIUBA - TA138")
+		(comment 1 "Lautaro, García Vitale - Padrón: 110028")
+		(comment 2 "Santiago Manuel, Cabrera - Padrón: 110445")
+		(comment 3 "Francisco Javier, Moya - Padrón: 109899")
+		(comment 4 "Integrantes:")
+	)
 	(junction
 		(at 123.19 46.99)
@@
 		)
 		(instances
-			(project "probando"
+			(project "esquematico"
 				(path "/70816206-2001-4ff4-9567-5d4a4798dbfa"
 					(reference "Q4")
@@
 		)
 		(instances
-			(project "probando"
+			(project "esquematico"
 				(path "/70816206-2001-4ff4-9567-5d4a4798dbfa"
 					(reference "Q3")
@@
 		)
 		(instances
-			(project "probando"
+			(project "esquematico"
 				(path "/70816206-2001-4ff4-9567-5d4a4798dbfa"
 					(reference "Q6")
@@
 		)
 		(instances
-			(project "probando"
+			(project "esquematico"
 				(path "/70816206-2001-4ff4-9567-5d4a4798dbfa"
 					(reference "#PWR02")
@@
 		)
 		(instances
-			(project "probando"
+			(project "esquematico"
 				(path "/70816206-2001-4ff4-9567-5d4a4798dbfa"
 					(reference "U2")
@@
 		)
 		(instances
-			(project "probando"
+			(project "esquematico"
 				(path "/70816206-2001-4ff4-9567-5d4a4798dbfa"
 					(reference "Q10")
@@
 		)
 		(instances
-			(project "probando"
+			(project "esquematico"
 				(path "/70816206-2001-4ff4-9567-5d4a4798dbfa"
 					(reference "Q5")
@@
 		)
 		(instances
-			(project "probando"
+			(project "esquematico"
 				(path "/70816206-2001-4ff4-9567-5d4a4798dbfa"
 					(reference "Q2")
@@
 		)
 		(instances
-			(project "probando"
+			(project "esquematico"
 				(path "/70816206-2001-4ff4-9567-5d4a4798dbfa"
 					(reference "R2")
@@
 		)
 		(instances
-			(project "probando"
+			(project "esquematico"
 				(path "/70816206-2001-4ff4-9567-5d4a4798dbfa"
 					(reference "R5")
@@
 		)
 		(instances
-			(project "probando"
+			(project "esquematico"
 				(path "/70816206-2001-4ff4-9567-5d4a4798dbfa"
 					(reference "#PWR01")
@@
 		)
 		(instances
-			(project "probando"
+			(project "esquematico"
 				(path "/70816206-2001-4ff4-9567-5d4a4798dbfa"
 					(reference "R8")
@@
 		)
 		(instances
-			(project "probando"
+			(project "esquematico"
 				(path "/70816206-2001-4ff4-9567-5d4a4798dbfa"
 					(reference "R9")
@@
 		)
 		(instances
-			(project "probando"
+			(project "esquematico"
 				(path "/70816206-2001-4ff4-9567-5d4a4798dbfa"
 					(reference "#PWR06")
@@
 		)
 		(instances
-			(project "probando"
+			(project "esquematico"
 				(path "/70816206-2001-4ff4-9567-5d4a4798dbfa"
 					(reference "#PWR03")
@@
 		)
 		(instances
-			(project "probando"
+			(project "esquematico"
 				(path "/70816206-2001-4ff4-9567-5d4a4798dbfa"
 					(reference "RL")
@@
 		)
 		(instances
-			(project "probando"
+			(project "esquematico"
 				(path "/70816206-2001-4ff4-9567-5d4a4798dbfa"
 					(reference "U1")
@@
 		)
 		(instances
-			(project "probando"
+			(project "esquematico"
 				(path "/70816206-2001-4ff4-9567-5d4a4798dbfa"
 					(reference "#PWR04")
@@
 		)
 		(instances
-			(project "probando"
+			(project "esquematico"
 				(path "/70816206-2001-4ff4-9567-5d4a4798dbfa"
 					(reference "J2")
@@
 		)
 		(instances
-			(project "probando"
+			(project "esquematico"
 				(path "/70816206-2001-4ff4-9567-5d4a4798dbfa"
 					(reference "JP3")
@@
 		)
 		(instances
-			(project "probando"
+			(project "esquematico"
 				(path "/70816206-2001-4ff4-9567-5d4a4798dbfa"
 					(reference "#PWR05")
@@
 		)
 		(instances
-			(project "probando"
+			(project "esquematico"
 				(path "/70816206-2001-4ff4-9567-5d4a4798dbfa"
 					(reference "Q9")
@@
 		)
 		(instances
-			(project "probando"
+			(project "esquematico"
 				(path "/70816206-2001-4ff4-9567-5d4a4798dbfa"
 					(reference "JP2")
@@
 		)
 		(instances
-			(project "probando"
+			(project "esquematico"
 				(path "/70816206-2001-4ff4-9567-5d4a4798dbfa"
 					(reference "R3")
@@
 		)
 		(instances
-			(project "probando"
+			(project "esquematico"
 				(path "/70816206-2001-4ff4-9567-5d4a4798dbfa"
 					(reference "JP1")
@@
 		)
 		(instances
-			(project "probando"
+			(project "esquematico"
 				(path "/70816206-2001-4ff4-9567-5d4a4798dbfa"
 					(reference "Q7")
@@
 		)
 		(instances
-			(project "probando"
+			(project "esquematico"
 				(path "/70816206-2001-4ff4-9567-5d4a4798dbfa"
 					(reference "R2")
@@
 		)
 		(instances
-			(project "probando"
+			(project "esquematico"
 				(path "/70816206-2001-4ff4-9567-5d4a4798dbfa"
 					(reference "Q8")
@@
 		)
 		(instances
-			(project "probando"
+			(project "esquematico"
 				(path "/70816206-2001-4ff4-9567-5d4a4798dbfa"
 					(reference "R4")
@@
 		)
 		(instances
-			(project "probando"
+			(project "esquematico"
 				(path "/70816206-2001-4ff4-9567-5d4a4798dbfa"
 					(reference "R1")
@@
 		)
 		(instances
-			(project "probando"
+			(project "esquematico"
 				(path "/70816206-2001-4ff4-9567-5d4a4798dbfa"
 					(reference "J1")
@@
 		)
 		(instances
-			(project "probando"
+			(project "esquematico"
 				(path "/70816206-2001-4ff4-9567-5d4a4798dbfa"
 					(reference "R7")
@@
 		)
 		(instances
-			(project "probando"
+			(project "esquematico"
 				(path "/70816206-2001-4ff4-9567-5d4a4798dbfa"
 					(reference "RS")
@@
 		)
 		(instances
-			(project "probando"
+			(project "esquematico"
 				(path "/70816206-2001-4ff4-9567-5d4a4798dbfa"
 					(reference "JP4")
@@
 		)
 		(instances
-			(project "probando"
+			(project "esquematico"
 				(path "/70816206-2001-4ff4-9567-5d4a4798dbfa"
 					(reference "R1")
@@
 		)
 		(instances
-			(project "probando"
+			(project "esquematico"
 				(path "/70816206-2001-4ff4-9567-5d4a4798dbfa"
 					(reference "R4")
@@
 		)
 		(instances
-			(project "probando"
+			(project "esquematico"
 				(path "/70816206-2001-4ff4-9567-5d4a4798dbfa"
 					(reference "JP5")

Commit message: 19.54
Other:
- title: Fuente Regulada con Protección Foldback -> Fuente Regulada con Protección Foldback - Grupo 5
Changed lines of the file:
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@@
 	(paper "A4")
 	(title_block
-		(title "Fuente Regulada con Protección Foldback")
+		(title "Fuente Regulada con Protección Foldback - Grupo 5")
 		(date "2026-04-10")
 		(company "FIUBA - TA138")

Commit message: Arreglando cosas
Parts:
- R3: value 4k4 -> 4k7
- R4: value 1k -> 680
Changed lines of the file:
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@@
 			)
 		)
-		(property "Value" "4k4"
+		(property "Value" "4k7"
 			(at 77.47 106.6799 0)
 			(show_name no)
@@
 			)
 		)
-		(property "Value" "1k"
+		(property "Value" "680"
 			(at 92.71 82.5499 0)
 			(show_name no)

Commit message: seguimos
Parts:
- added R12, R13: 10k, symbol Device:R
Connections:
- net GND: now also R12.2
- net at JP4.2 (B), U2.1: now also R13.2
- net at R8.2, R9.1, U2.2 (-): now also R13.1
- net at R7.2, U2.3 (+): now also R12.1
Other:
- moved on the sheet: R7, R8, RS, U2A
