File: Checkpoint 5/KiCAD/switching_v1/switching_v1.kicad_sch (KiCad schematic)
At the start: 27 parts, among them J1 Conn_01x02, J2 Conn_01x02, U1 LM7809_TO220, U2 LM393, U4 TL072

Commit message: avances CP5
Parts:
- removed J2: Conn_01x02, TerminalBlock:TerminalBlock_MaiXu_MX126-5.0-02P_1x02_P5.00mm, symbol Connector_Generic:Conn_01x02
- added C10, C14, C7, C8: 0.1u, Capacitor_THT:C_Disc_D5.0mm_W2.5mm_P2.50mm, symbol Device:C
- added C11, C12, C13, C6: C, Capacitor_THT:C_Disc_D5.0mm_W2.5mm_P2.50mm, symbol Device:C
- added C3, C4: C_Polarized, symbol Device:C_Polarized
- added C9: 1u, Capacitor_THT:C_Disc_D5.0mm_W2.5mm_P2.50mm, symbol Device:C
- added D1, D2, D4: D_Schottky, Diode_THT:D_DO-15_P15.24mm_Horizontal, symbol Device:D_Schottky
- added D3: LED, LED_THT:LED_D5.0mm_IRGrey, symbol Device:LED
- added J3: Conn_01x02, TerminalBlock:TerminalBlock_MaiXu_MX126-5.0-02P_1x02_P5.00mm, symbol Connector_Generic:Conn_01x02
- added L1: L, symbol Device:L
- added Q1, Q2: IRF740, Package_TO_SOT_THT:TO-220-3_Vertical, symbol Transistor_FET:IRF740
- added R10, R7, R8: 1, Resistor_THT:R_Axial_DIN0207_L6.3mm_D2.5mm_P7.62mm_Horizontal, symbol Device:R
- added R12, R13, R14, R3: R, Resistor_THT:R_Axial_DIN0207_L6.3mm_D2.5mm_P7.62mm_Horizontal, symbol Device:R
- added TP8, TP9: TestPoint, Connector_PinHeader_2.54mm:PinHeader_1x01_P2.54mm_Vertical, symbol Connector:TestPoint
- added unit 3 of U2
- added U3: IR2104, Package_DIP:DIP-8_W7.62mm_LongPads, symbol Driver_FET:IR2104
- added unit 3 of U4
- added U5: TL071, Package_DIP:DIP-8_W7.62mm_LongPads, symbol Amplifier_Operational:TL071
- R11: value 0 -> R
- TP1, TP2, TP3: footprint (none) -> Connector_PinHeader_2.54mm:PinHeader_1x01_P2.54mm_Vertical
- TP5: value TestPoint -> TP-Switching
Connections:
- net +9V: now also C14.1, C7.1, C8.1, C9.2, R10.1, U2.8 (V+), U3.1 (VCC), U4.8 (V+), U5.7 (V+)
- net +BATT: now also C3.1, D1.1 (K), Q1.2 (D), TP8.1
- net GND: now also R11.2, C10.2, C14.2, C3.2, C4.2, C6.2, C7.2, C8.2, C9.1, D1.2 (A), D2.1 (K), D2.2 (A), D3.1 (K), J3.2 (Pin_2), L1.1, Q1.3 (S), Q2.2 (D), Q2.3 (S), TP9.1, U2.4 (V-), U3.4 (COM), U3.6 (VS), U4.4 (V-), U5.1 (NULL), U5.4 (V-), U5.5 (NULL)
- net PWM: now also U3.2 (IN)
- net Vref: now also U4.5 (+); no longer R11.1
- removed net Vref_opamp: R11.2, U4.5 (+)
- new net: R7.1, U3.5 (LO)
- new net: D4.2 (A), R10.2
- new net: D3.2 (A), R3.2
- new net: R8.1, U3.7 (HO)
- new net: C10.1, D4.1 (K), U3.8 (VB)
- new net: C12.2, C13.2, R11.1, R12.1, R13.1, U5.2 (-)
- new net: C11.1, R13.2
- new net: C12.1, R14.2
- new net: C13.1, R14.1, U5.6
- new net HO: Q1.1 (G), R8.2
- new net LO: Q2.1 (G), R7.2
- new net Vo: C11.2, C4.1, C6.1, J3.1 (Pin_1), L1.2, R12.2, R3.1
- new net Vref_comp: U5.3 (+)
Other:
- note added: "Faltan: - Referencia de tensión en la compensación + adaptar la salida de la compensación a la entrada del PWM - Entrada SD del IR2104 + Corregir los valores de los componentes -elegir una huella para C3 (depende de qué tan grande sea)"
- moved on the sheet: C1, C2, C5, JP1, JP2, JP3, JP4, R1, R2, R5, R6, R9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

Commit message: avances PCB
Parts:
- added C15: C_Polarized, Capacitor_THT:CP_Radial_D10.0mm_P5.00mm, symbol Device:C_Polarized
- added JP5: SD_IN, Connector_PinHeader_2.54mm:PinHeader_1x02_P2.54mm_Vertical, symbol Jumper:Jumper_2_Bridged
- added R15: 5k1, Resistor_THT:R_Axial_DIN0207_L6.3mm_D2.5mm_P7.62mm_Horizontal, symbol Device:R
- added TP10: TestPoint, Connector_PinHeader_2.54mm:PinHeader_1x01_P2.54mm_Vertical, symbol Connector:TestPoint
- C3: footprint (none) -> Capacitor_THT:CP_Radial_D10.0mm_P5.00mm
- C5: value 33p -> 56p
- L1: footprint (none) -> Transformer_THT:Transformer_37x44
- R11: value R -> 56k
- R5: value 150k -> 220k
Connections:
- net Vref_comp is gone; now on net Vref: U5.3 (+)
- net +9V: now also JP5.1 (A)
- net +BATT: now also C15.1
- net GND: now also C15.2, R15.2; no longer R11.2
- net PWM_ref: now also C13.1, R14.1, U5.6, TP10.1
- net at U3.3 (~{SD}): now also JP5.2 (B)
- new net: R11.2, R15.1
Other:
- note added: "Faltan: + Corregir los valores de los componentes 1)PWM 2)compensación 3)buck"
- note added: "NOTA: Los componentes del integrador también pueden ser R = 120k y C = 100p (por si no se consiguen)"
- note removed: "Faltan: - Referencia de tensión en la compensación + adaptar la salida de la compensación a la entrada del PWM - Entrada SD del IR2104 + Corregir los valores de los componentes -elegir una huella para C3 (depende de qué tan grande sea)"
- moved on the sheet: C14

Commit message: Avances PCB
Parts:
- removed TP1, TP2, TP3, TP4: TestPoint, Connector_PinHeader_2.54mm:PinHeader_1x01_P2.54mm_Vertical, symbol Connector:TestPoint
- added JP10: TP_Bootstrap, Connector_PinHeader_2.54mm:PinHeader_1x02_P2.54mm_Vertical, symbol Jumper:Jumper_2_Bridged
- added JP6: TP_PWM, Connector_PinHeader_2.54mm:PinHeader_1x02_P2.54mm_Vertical, symbol Jumper:Jumper_2_Bridged
- added JP7, JP9: TP_Vc, Connector_PinHeader_2.54mm:PinHeader_1x02_P2.54mm_Vertical, symbol Jumper:Jumper_2_Bridged
- added JP8: TP_HO, Connector_PinHeader_2.54mm:PinHeader_1x02_P2.54mm_Vertical, symbol Jumper:Jumper_2_Bridged
- C15, C3: value C_Polarized -> 330u
- C4: value C_Polarized -> 10u; footprint (none) -> Capacitor_THT:CP_Radial_D5.0mm_P2.50mm
- C6: value C -> 1n; footprint Capacitor_THT:C_Disc_D5.0mm_W2.5mm_P2.50mm -> Capacitor_THT:C_Disc_D14.5mm_W5.0mm_P10.00mm
- Cc1: renamed from C12; value C -> 22n
- Cc2: renamed from C11; value C -> 1.2n
- Cc3: renamed from C13; value C -> 5.6n
- D1, D2, D4: footprint Diode_THT:D_DO-15_P15.24mm_Horizontal -> Diode_THT:D_DO-201AD_P12.70mm_Horizontal
- JP2: value Jumper_2_Bridged -> TP_Cuadrada
- JP3: value Jumper_2_Bridged -> TP_Traing
- JP4: value Jumper_2_Bridged -> Jumper_9V
- L1: value L -> 427u
- R3: value R -> 4k7
- Rc1: renamed from R12; value R -> 68k
- Rc2: renamed from R14; value R -> 3k3
- Rc3: renamed from R13; value R -> 680
- TP10: value TestPoint -> TP_Vo
- TP5: value TP-Switching -> TP_Sw
- TP8, TP9: footprint Connector_PinHeader_2.54mm:PinHeader_1x01_P2.54mm_Vertical -> Connector_PinHeader_2.54mm:PinHeader_1x02_P2.54mm_Vertical
Connections:
- net GND: no longer C10.2, D1.2 (A), D2.1 (K), L1.1, Q1.3 (S), Q2.2 (D), TP5.1, U3.6 (VS)
- net HO: now also JP8.1 (A); no longer Q1.1 (G)
- net LO: now also JP9.1 (A); no longer Q2.1 (G)
- net PWM: now also JP6.1 (A); no longer U3.2 (IN)
- net PWM_ref: now also JP7.1 (A); no longer Cc3.1, Rc2.1, TP10.1, U5.6
- net Vo: now also TP10.1
- net at C10.1, U3.8 (VB): now also JP10.2 (B); no longer D4.1 (K)
- new net: D4.1 (K), JP10.1 (A)
- new net: Cc3.1, JP7.2 (B), Rc2.1, U5.6
- new net GH: JP8.2 (B), Q1.1 (G)
- new net GL: JP9.2 (B), Q2.1 (G)
- new net PWM_out: JP6.2 (B), U3.2 (IN)
- new net SW: C10.2, D1.2 (A), D2.1 (K), L1.1, Q1.3 (S), Q2.2 (D), TP5.1, U3.6 (VS)
Other:
- note added: "Test points importantes: 1)nodo switching (sw) 2) gates de los MOSFET 3) Nodo de salida 4) Alimentación (BAT y GND). Poner pines para que la conección sea más cómoda 5) Tensión de control Vc 6) Cuadrada 7) traingular 8)PWM 9) Capacitor de Bootstrap"
- note removed: "Faltan: + Corregir los valores de los componentes 1)PWM 2)compensación 3)buck"
- moved on the sheet: C4, C6, D3, D4, JP2, L1, R10, R3
