File: Checkpoint 5/KiCAD/switching_v1/switching_v1.kicad_pcb (KiCad board)
At the start: 2 copper layers, 24 parts, among them J1 Conn_01x02, J2 Conn_01x02, U1 LM7809_TO220, U2 LM393, U4 TL072

Commit message: avances PCB
Parts:
- added C10: 0.1u, Capacitor_THT:C_Disc_D5.0mm_W2.5mm_P2.50mm, F.Cu at (149.9, 81.3)
- added C11: C, Capacitor_THT:C_Disc_D5.0mm_W2.5mm_P2.50mm, F.Cu at (149.9, 85.4)
- added C12: C, Capacitor_THT:C_Disc_D5.0mm_W2.5mm_P2.50mm, F.Cu at (149.9, 89.4)
- added C13: C, Capacitor_THT:C_Disc_D5.0mm_W2.5mm_P2.50mm, F.Cu at (149.9, 93.5)
- added C14: 0.1u, Capacitor_THT:C_Disc_D5.0mm_W2.5mm_P2.50mm, F.Cu at (149.9, 97.5)
- added C15: C_Polarized, Capacitor_THT:CP_Radial_D10.0mm_P5.00mm, F.Cu at (106.7, 120.1)
- added C3: C_Polarized, Capacitor_THT:CP_Radial_D10.0mm_P5.00mm, F.Cu at (106.7, 108.5)
- added C6: C, Capacitor_THT:C_Disc_D5.0mm_W2.5mm_P2.50mm, F.Cu at (149.9, 65.1)
- added C7: 0.1u, Capacitor_THT:C_Disc_D5.0mm_W2.5mm_P2.50mm, F.Cu at (149.9, 69.2)
- added C8: 0.1u, Capacitor_THT:C_Disc_D5.0mm_W2.5mm_P2.50mm, F.Cu at (149.9, 73.2)
- added C9: 1u, Capacitor_THT:C_Disc_D5.0mm_W2.5mm_P2.50mm, F.Cu at (149.9, 77.3)
- added D1: D_Schottky, Diode_THT:D_DO-15_P15.24mm_Horizontal, F.Cu at (126.1, 105.3)
- added D2: D_Schottky, Diode_THT:D_DO-15_P15.24mm_Horizontal, F.Cu at (126.1, 110.5)
- added D3: LED, LED_THT:LED_D5.0mm_IRGrey, F.Cu at (126.6, 121.9)
- added D4: D_Schottky, Diode_THT:D_DO-15_P15.24mm_Horizontal, F.Cu at (126.1, 115.6)
- added J3: Conn_01x02, TerminalBlock:TerminalBlock_MaiXu_MX126-5.0-02P_1x02_P5.00mm, F.Cu at (158.9, 107.8)
- added JP5: SD_IN, Connector_PinHeader_2.54mm:PinHeader_1x02_P2.54mm_Vertical, F.Cu at (133.9, 120.5)
- added L1: L, Transformer_THT:Transformer_37x44, F.Cu at (117.9, 70.2)
- added Q1: IRF740, Package_TO_SOT_THT:TO-220-3_Vertical, F.Cu at (146.6, 106.7)
- added Q2: IRF740, Package_TO_SOT_THT:TO-220-3_Vertical, F.Cu at (146.6, 112.6)
- added R10: 1, Resistor_THT:R_Axial_DIN0207_L6.3mm_D2.5mm_P7.62mm_Horizontal, F.Cu at (156.0, 77.3)
- added R11: 56k, Resistor_THT:R_Axial_DIN0207_L6.3mm_D2.5mm_P7.62mm_Horizontal, F.Cu at (156.0, 81.3)
- added R12: R, Resistor_THT:R_Axial_DIN0207_L6.3mm_D2.5mm_P7.62mm_Horizontal, F.Cu at (156.0, 85.4)
- added R13: R, Resistor_THT:R_Axial_DIN0207_L6.3mm_D2.5mm_P7.62mm_Horizontal, F.Cu at (156.0, 89.4)
- added R14: R, Resistor_THT:R_Axial_DIN0207_L6.3mm_D2.5mm_P7.62mm_Horizontal, F.Cu at (156.0, 93.5)
- added R15: 5k1, Resistor_THT:R_Axial_DIN0207_L6.3mm_D2.5mm_P7.62mm_Horizontal, F.Cu at (156.0, 97.5)
- added R3: R, Resistor_THT:R_Axial_DIN0207_L6.3mm_D2.5mm_P7.62mm_Horizontal, F.Cu at (156.0, 65.1)
- added R7: 1, Resistor_THT:R_Axial_DIN0207_L6.3mm_D2.5mm_P7.62mm_Horizontal, F.Cu at (156.0, 69.2)
- added R8: 1, Resistor_THT:R_Axial_DIN0207_L6.3mm_D2.5mm_P7.62mm_Horizontal, F.Cu at (156.0, 73.2)
- added TP1: TestPoint, Connector_PinHeader_2.54mm:PinHeader_1x01_P2.54mm_Vertical, F.Cu at (117.3, 105.0)
- added TP10: TestPoint, Connector_PinHeader_2.54mm:PinHeader_1x01_P2.54mm_Vertical, F.Cu at (121.9, 114.2)
- added TP2: TestPoint, Connector_PinHeader_2.54mm:PinHeader_1x01_P2.54mm_Vertical, F.Cu at (117.3, 109.6)
- added TP3: TestPoint, Connector_PinHeader_2.54mm:PinHeader_1x01_P2.54mm_Vertical, F.Cu at (117.3, 114.2)
- added TP5: TP-Switching, Connector_PinHeader_2.54mm:PinHeader_1x01_P2.54mm_Vertical, F.Cu at (117.3, 118.8)
- added TP8: TestPoint, Connector_PinHeader_2.54mm:PinHeader_1x01_P2.54mm_Vertical, F.Cu at (121.9, 105.0)
- added TP9: TestPoint, Connector_PinHeader_2.54mm:PinHeader_1x01_P2.54mm_Vertical, F.Cu at (121.9, 109.6)
- added U3: IR2104, Package_DIP:DIP-8_W7.62mm_LongPads, F.Cu at (145.3, 116.7)
- added U5: TL071, Package_DIP:DIP-8_W7.62mm_LongPads, F.Cu at (156.9, 116.7)
- C5: value 33p -> 56p
- R5: value 150k -> 220k
- moved J1 79.2 mm to (197.0, 85.1)
- moved R1 79.2 mm to (183.7, 82.1)
- moved R11 79.2 mm to (183.7, 102.4)
- moved R6 79.2 mm to (183.7, 94.3)
- moved C1 79.2 mm to (212.1, 82.1)
- moved R5 79.2 mm to (183.7, 90.2)
- moved R9 79.2 mm to (183.7, 98.3)
- moved Rf2 79.2 mm to (183.7, 110.5)
- moved U2 79.2 mm to (195.0, 102.4)
- moved U4 79.2 mm to (206.7, 102.4)
- moved J2 79.2 mm to (197.0, 95.2)
- moved R2 79.2 mm to (183.7, 86.2)
- moved Rf1 79.2 mm to (183.7, 106.4)
- moved C2 79.2 mm to (212.1, 86.2)
- moved C5 79.2 mm to (212.1, 90.2)
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Connections:
- U2 pad 4: (no net) -> GND
- U2 pad 8: (no net) -> +9V
- U4 pad 4: (no net) -> GND
- U4 pad 5: /Vref_opamp -> /Vref
- U4 pad 8: (no net) -> +9V
Other:
- board outline added: 147 x 92.1 mm

Commit message: Avances PCB
Parts:
- removed J2: Conn_01x02, TerminalBlock:TerminalBlock_MaiXu_MX126-5.0-02P_1x02_P5.00mm
- removed the TP5 at (207.8, 87.0)
- added C4: 10u, Capacitor_THT:CP_Radial_D5.0mm_P2.50mm, F.Cu at (110.0, 148.0)
- added JP10: TP_Bootstrap, Connector_PinHeader_2.54mm:PinHeader_1x02_P2.54mm_Vertical, F.Cu at (123.5, 104.2)
- added JP6: TP_PWM, Connector_PinHeader_2.54mm:PinHeader_1x02_P2.54mm_Vertical, F.Cu at (150.5, 67.0)
- added JP7: TP_Vc, Connector_PinHeader_2.54mm:PinHeader_1x02_P2.54mm_Vertical, F.Cu at (141.0, 118.0)
- added JP8: TP_HO, Connector_PinHeader_2.54mm:PinHeader_1x02_P2.54mm_Vertical, F.Cu at (106.7, 89.1)
- added JP9: TP_Vc, Connector_PinHeader_2.54mm:PinHeader_1x02_P2.54mm_Vertical, F.Cu at (106.7, 82.7)
- C15, C3: value C_Polarized -> 330u
- C6: value C -> 1n; footprint Capacitor_THT:C_Disc_D5.0mm_W2.5mm_P2.50mm -> Capacitor_THT:C_Disc_D14.5mm_W5.0mm_P10.00mm
- Cc1: renamed from C12; value C -> 22n
- Cc2: renamed from C11; value C -> 1.2n
- Cc3: renamed from C13; value C -> 5.6n
- D1, D2, D4: footprint Diode_THT:D_DO-15_P15.24mm_Horizontal -> Diode_THT:D_DO-201AD_P12.70mm_Horizontal
- JP2: value Jumper_2_Bridged -> TP_Cuadrada
- JP3: value Jumper_2_Bridged -> TP_Traing
- JP4: value Jumper_2_Bridged -> Jumper_9V
- L1: value L -> 427u
- R3: value R -> 4k7
- Rc1: renamed from R12; value R -> 68k
- Rc2: renamed from R14; value R -> 3k3
- Rc3: renamed from R13; value R -> 680
- TP10: value TestPoint -> TP_Vo
- TP5: value TP-Switching -> TP_Sw
- TP8, TP9: footprint Connector_PinHeader_2.54mm:PinHeader_1x01_P2.54mm_Vertical -> Connector_PinHeader_2.54mm:PinHeader_1x02_P2.54mm_Vertical
- moved C14 184.8 mm to (332.9, 123.5)
- moved C7 184.8 mm to (332.9, 95.2)
- moved Cc1 184.8 mm to (332.9, 115.4)
- moved Cc2 184.8 mm to (332.9, 111.4)
- moved Cc3 184.8 mm to (332.9, 119.5)
- moved J3 184.8 mm to (341.9, 133.8)
- moved JP1 184.8 mm to (378.2, 140.5)
- moved R11 184.8 mm to (366.7, 128.4)
- moved TP3 184.8 mm to (300.3, 140.2)
- moved TP9 184.8 mm to (304.9, 135.6)
- moved R11 184.8 mm to (339.0, 107.3)
- moved R15 184.8 mm to (339.0, 123.5)
- moved Rc2 184.8 mm to (339.0, 119.5)
- moved Rc3 184.8 mm to (339.0, 115.4)
- moved TP4 184.8 mm to (390.8, 108.4)
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Connections:
- C10 pad 1: Net-(D4-K) -> Net-(JP10-B)
- C10 pad 2: GND -> /SW
- Cc3 pad 1: /PWM_ref -> Net-(JP7-B)
- D1 pad 2: GND -> /SW
- D2 pad 1: GND -> /SW
- L1 pad 1: GND -> /SW
- Q1 pad 1: /HO -> /GH
- Q1 pad 3: GND -> /SW
- Q2 pad 1: /LO -> /GL
- Q2 pad 2: GND -> /SW
- Rc2 pad 1: /PWM_ref -> Net-(JP7-B)
- TP10 pad 1: /PWM_ref -> /Vo
- TP5 pad 1: GND -> /SW
- U3 pad 2: /PWM -> /PWM_out
- U3 pad 6: GND -> /SW
- U3 pad 8: Net-(D4-K) -> Net-(JP10-B)
- U5 pad 6: /PWM_ref -> Net-(JP7-B)
Routing:
- net /SW: track 0.00 -> 64.8 mm
- net /PWM_ref: track 0.00 -> 57.2 mm
- net /Triang: track 0.00 -> 50.0 mm
- net /PWM_out: track 0.00 -> 33.2 mm
- net /Cuad: track 0.00 -> 29.5 mm
- net Net-(JP5-B): track 0.00 -> 21.9 mm, vias 0 -> 2
- net Net-(JP3-B): track 0.00 -> 19.7 mm
- net /PWM: track 0.00 -> 19.1 mm
- net Net-(JP10-B): track 0.00 -> 14.5 mm
- net /Vo: track 0.00 -> 13.4 mm
- net Net-(U4B--): track 0.00 -> 11.4 mm
- net Net-(JP7-B): track 0.00 -> 11.1 mm
- net +9V: track 0.00 -> 10.8 mm
- net Net-(U2A-+): track 0.00 -> 7.67 mm
- net Net-(D4-K): track 0.00 -> 5.51 mm
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- added copper zone on B.Cu, net +BATT
Other:
- board size 147 x 92.1 mm -> 200 x 130 mm

Commit message: correción PCB
Parts:
- removed the R11 at (366.7, 128.4)
- removed TP1, TP2, TP3, TP4, TP6, TP7: TestPoint, Connector_PinHeader_2.54mm:PinHeader_1x01_P2.54mm_Vertical
- removed TP8, TP9: TestPoint, Connector_PinHeader_2.54mm:PinHeader_1x02_P2.54mm_Vertical
- added J2: TP_BATT, Connector_PinHeader_2.54mm:PinHeader_1x02_P2.54mm_Vertical, F.Cu at (61.5, 43.0)
- added J4: TP_GND, Connector_PinHeader_2.54mm:PinHeader_1x02_P2.54mm_Vertical, F.Cu at (89.5, 43.2)
- added J5: TP_GND, Connector_PinHeader_2.54mm:PinHeader_1x02_P2.54mm_Vertical, F.Cu at (98.5, 111.8)
- moved JP1 276.0 mm to (120.3, 42.0), turned to -90 degrees
- moved J3 225.4 mm to (117.0, 148.2)
- moved Cc2 195.7 mm to (139.5, 141.2), turned to 180 degrees
- moved C7 195.4 mm to (140.5, 61.0)
- moved Rc3 189.7 mm to (151.1, 141.2), turned to 180 degrees
- moved Cc1 188.7 mm to (145.5, 137.0), turned to 180 degrees
- moved C14 184.5 mm to (148.5, 127.2)
- moved Rc2 183.1 mm to (156.8, 137.0), turned to 180 degrees
- moved R11 174.9 mm to (167.5, 141.3), turned to 90 degrees
- moved Cc3 173.0 mm to (161.0, 138.5), turned to -90 degrees
- moved R15 171.7 mm to (167.5, 131.0), turned to 180 degrees
- moved R3 13.0 mm to (110.0, 148.3)
- moved D3 13.0 mm to (110.0, 133.0)
- moved R9 7.38 mm to (150.5, 70.5)
- moved C4 6.75 mm to (103.2, 148.2)
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Routing:
- net Net-(U5--): track 4.45 -> 47.7 mm
- net GND: track 0.00 -> 26.1 mm
- net Net-(JP7-B): track 11.1 -> 36.6 mm
- net +9V: track 10.8 -> 30.6 mm
- net Net-(JP1-A): track 0.00 -> 8.27 mm
- net /PWM_out: track 33.2 -> 26.7 mm
- net /Vo: track 13.4 -> 18.2 mm
- net Net-(Cc2-Pad1): track 0.00 -> 3.94 mm
- net Net-(Cc1-Pad1): track 0.00 -> 3.69 mm
- net Net-(R11-Pad2): track 0.00 -> 2.69 mm
- net /PWM: track 19.1 -> 21.3 mm
