File: Checkpoint 5/KiCAD/switching_v2/switching_v2.kicad_sch (KiCad schematic)
At the start: 60 parts, among them J1 Conn_01x02, J2 TP_BATT, J3 Conn_01x02, J4 TP_GND, J5 TP_GND, Q1 IRF740, Q2 IRF740, U1 LM7809_TO220, U2 LM393, U3 IR2104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

Commit message: correción PCB
Parts:
- removed JP1: Jumper_2_Bridged, Connector_PinHeader_2.54mm:PinHeader_1x02_P2.54mm_Vertical, symbol Jumper:Jumper_2_Bridged
- removed JP10: TP_Bootstrap, Connector_PinHeader_2.54mm:PinHeader_1x02_P2.54mm_Vertical, symbol Jumper:Jumper_2_Bridged
- removed JP2: TP_Cuadrada, Connector_PinHeader_2.54mm:PinHeader_1x02_P2.54mm_Vertical, symbol Jumper:Jumper_2_Bridged
- removed JP3: TP_Traing, Connector_PinHeader_2.54mm:PinHeader_1x02_P2.54mm_Vertical, symbol Jumper:Jumper_2_Bridged
- removed U5: TL071, Package_DIP:DIP-8_W7.62mm_LongPads, symbol Amplifier_Operational:TL071
- added J6: TP_Cuad, Connector_PinHeader_2.54mm:PinHeader_1x02_P2.54mm_Vertical, symbol Connector:Conn_01x02_Pin
- added J7: TP_Triang, Connector_PinHeader_2.54mm:PinHeader_1x02_P2.54mm_Vertical, symbol Connector:Conn_01x02_Pin
- added J8: TP_Bootstrap, Connector_PinHeader_2.54mm:PinHeader_1x02_P2.54mm_Vertical, symbol Connector:Conn_01x02_Pin
- added R12, R4: 470k, Resistor_THT:R_Axial_DIN0207_L6.3mm_D2.5mm_P7.62mm_Horizontal, symbol Device:R
- added U6: TL072, Package_DIP:DIP-8_W7.62mm_Socket_LongPads, symbol Amplifier_Operational:TL072
- R7, R8: footprint Resistor_THT:R_Axial_DIN0207_L6.3mm_D2.5mm_P7.62mm_Horizontal -> Resistor_THT:R_Axial_DIN0309_L9.0mm_D3.2mm_P15.24mm_Horizontal
Connections:
- net +9V: now also D4.2 (A), R4.1, U6.8 (V+); no longer R10.1
- net Cuad: now also R5.1, J6.1 (Pin_1), J6.2 (Pin_2)
- net GND: now also R12.2, U6.4 (V-)
- net Triang: now also U2.6 (-), J7.1 (Pin_1), J7.2 (Pin_2)
- net Vo: now also Rc3.2; no longer Cc2.2
- net Vref: now also U4.1, U4.2 (-)
- net at D4.1 (K): now also R10.1
- net at C10.1, U3.8 (VB): now also R10.2, J8.1 (Pin_1), J8.2 (Pin_2)
- net at Cc3.1, JP7.2 (B), Rc2.1: now also U6.1
- net at Cc1.2, Cc3.2, R11.1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: now also Cc2.1, U6.2 (-); no longer Rc3.1
- new net: R12.1, R4.2, U6.5 (+)
- new net: Cc2.2, Rc3.1
- new net Vref_comp: U6.3 (+), U6.6 (-), U6.7
Other:
- moved on the sheet: C14, Cc1, Cc2, Cc3, D4, J4, JP7, R10, R11, R15, Rc1, Rc2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
